File: Hardware/clock/clock.kicad_pcb (KiCad board)
At the start: 2 copper layers, 132.2 x 55 mm, 45 parts, among them J1 Barrel_Jack_Switch, J2 Conn_01x05_Pin, J3 Conn_02x03_Odd_Even, J4 Conn_01x02_Pin, J5 Conn_01x06_Pin, Q1 BC817, Q2 BC817, SW1 PTH_RA_h7.5mm, U1 SBC18-11EGWA, U2 SBC18-11EGWA, U3 SBC18-11EGWA, U4 ESP32-WROOM-32, U5 SBC18-11EGWA, U6 MAX7221xNG, U7 AMS1117-3.3, U8 LM2596S-5

Commit message: Refactor code structure for improved readability and maintainability
Routing:
- net /15: track 29.5 -> 24.9 mm
- net /2: track 12.0 -> 7.51 mm
- net GND: vias 19 -> 27
Changed lines of the file:
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@@
 	)
 	(via
+		(at 103.77 100.95)
+		(size 0.6)
+		(drill 0.3)
+		(layers "F.Cu" "B.Cu")
+		(free yes)
+		(net 1)
+	)
+	(via
 		(at 57.52 121.8475)
 		(size 0.6)
@@
 	)
 	(via
+		(at 100.28 100.91)
+		(size 0.6)
+		(drill 0.3)
+		(layers "F.Cu" "B.Cu")
+		(net 1)
+	)
+	(via
 		(at 169.65 110.14)
 		(size 0.6)
@@
 	)
 	(via
+		(at 102.71 100.93)
+		(size 0.6)
+		(drill 0.3)
+		(layers "F.Cu" "B.Cu")
+		(free yes)
+		(net 1)
+	)
+	(via
+		(at 99.08 102.21)
+		(size 0.6)
+		(drill 0.3)
+		(layers "F.Cu" "B.Cu")
+		(free yes)
+		(net 1)
+	)
+	(via
 		(at 81.5 116.8)
 		(size 0.6)
@@
 	)
 	(via
+		(at 99.11 100.88)
+		(size 0.6)
+		(drill 0.3)
+		(layers "F.Cu" "B.Cu")
+		(free yes)
+		(net 1)
+	)
+	(via
 		(at 56.62 121.8475)
 		(size 0.6)
@@
 	)
 	(via
+		(at 97.76 100.83)
+		(size 0.6)
+		(drill 0.3)
+		(layers "F.Cu" "B.Cu")
+		(free yes)
+		(net 1)
+	)
+	(via
+		(at 97.78 102.2)
+		(size 0.6)
+		(drill 0.3)
+		(layers "F.Cu" "B.Cu")
+		(free yes)
+		(net 1)
+	)
+	(via
+		(at 101.5 100.91)
+		(size 0.6)
+		(drill 0.3)
+		(layers "F.Cu" "B.Cu")
+		(free yes)
+		(net 1)
+	)
+	(via
 		(at 67.69 125.57)
 		(size 0.6)
@@
 	)
 	(segment
-		(start 149.68 107.07)
-		(end 149.68 108.25)
+		(start 149.83 108.4)
+		(end 149.83 107.22)
 		(width 0.2)
 		(layer "F.Cu")
@@
 	)
 	(segment
-		(start 152.68 109.9)
-		(end 154.28 111.5)
+		(start 151.9 111.26)
+		(end 151.9 110.47)
 		(width 0.2)
 		(layer "F.Cu")
@@
 	)
 	(segment
-		(start 151.33 109.9)
-		(end 152.68 109.9)
+		(start 151.9 110.47)
+		(end 149.83 108.4)
 		(width 0.2)
 		(layer "F.Cu")
@@
 	)
 	(segment
-		(start 149.34 106.73)
-		(end 149.68 107.07)
-		(width 0.2)
-		(layer "F.Cu")
-		(net 35)
-	)
-	(segment
-		(start 149.68 108.25)
-		(end 151.33 109.9)
+		(start 149.83 107.22)
+		(end 149.34 106.73)
 		(width 0.2)
 		(layer "F.Cu")
@@
 	)
 	(via
-		(at 154.28 111.5)
+		(at 151.9 111.26)
 		(size 0.6)
 		(drill 0.3)
@@
 	)
 	(segment
-		(start 154.28 111.5)
-		(end 154.04 111.26)
-		(width 0.2)
-		(layer "B.Cu")
-		(net 35)
-	)
-	(segment
-		(start 154.04 111.26)
-		(end 151.9 111.26)
-		(width 0.2)
-		(layer "B.Cu")
-		(net 35)
-	)
-	(segment
 		(start 129.05 115.01)
 		(end 128.99 114.95)
@@
 	)
 	(segment
-		(start 153.74 112.53)
-		(end 154.05 112.84)
-		(width 0.3)
-		(layer "F.Cu")
-		(net 48)
-	)
-	(segment
-		(start 143.91 107.59)
+		(start 151.9 112.53)
 		(end 148.85 112.53)
 		(width 0.3)
@@
 	(segment
 		(start 148.85 112.53)
-		(end 153.74 112.53)
+		(end 143.91 107.59)
 		(width 0.3)
 		(layer "F.Cu")
@@
 	)
 	(segment
-		(start 143.91 103.32)
-		(end 143.91 107.59)
+		(start 143.91 107.59)
+		(end 143.91 103.32)
 		(width 0.3)
 		(layer "F.Cu")
@@
 	)
 	(via
-		(at 154.05 112.84)
+		(at 151.9 112.53)
 		(size 0.6)
 		(drill 0.3)
@@
 	)
 	(segment
-		(start 154.05 112.84)
-		(end 153.74 112.53)
-		(width 0.3)
-		(layer "B.Cu")
-		(net 48)
-	)
-	(segment
 		(start 140.255 94.265)
 		(end 140.29 94.23)
@@
 		(width 0.3)
 		(layer "B.Cu")
-		(net 48)
-	)
-	(segment
-		(start 153.74 112.53)
-		(end 151.9 112.53)
-		(width 0.3)
-		(layer "B.Cu")
